File: downloader.sch (KiCad schematic (older format))
At the start: 16 parts, among them J1 USB_C_Receptacle_USB2.0, J2 Conn_01x06_Female, Q1 SS8050-G, Q2 SS8050-G, SW1 SW_Push, SW2 SW_Push, U1 AMS1117-3.3, U2 ch340k

Commit message: version2.0
Parts:
- added C3: 0.1uf, Capacitor_SMD:C_0603_1608Metric, symbol Device:C
- added C4: 0.1UF, Capacitor_SMD:C_0603_1608Metric, symbol Device:C
- added D2, D3: LED, Diode_SMD:D_0603_1608Metric, symbol Device:LED
- added R3, R5: 10k, Resistor_SMD:R_0603_1608Metric, symbol Device:R
- R1: value 470 -> 10k
- U2: footprint Package_SO:SSOP-10_3.9x4.9mm_P1.00mm -> my:ESSOP-10_3.9x4.9mm_P1.00mm
- renumbered C3 to C2, C2 to C5, C4 to C6, R3 to R4
Connections:
- net labels added: VCC
- wire segments 59 -> 72
- no-connect marks 5 -> 6
Other:
- moved on the sheet: C1, C2, C5, C6, D1, J1, J2, Q1, Q2, R1, R4, SW1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

Commit message: version2.0
Parts:
- removed C1, C2: 10uf, Capacitor_SMD:C_0603_1608Metric, symbol Device:C
- removed Q1, Q2: SS8050-G, Package_TO_SOT_SMD:SOT-23, symbol my:SS8050-G
- removed R4, R5: 10k, Resistor_SMD:R_0603_1608Metric, symbol Device:R
- removed U1: AMS1117-3.3, Package_TO_SOT_SMD:SOT-223-3_TabPin2, symbol Regulator_Linear:AMS1117-3.3
- added U1: DDC114TU-7-F, Package_TO_SOT_SMD:SOT-363_SC-70-6, symbol my:DDC114TU-7-F
Connections:
- net labels removed: +3.3V
- wire segments 72 -> 57
Other:
- moved on the sheet: C3, C4, C5, C6, D2, D3, R2, R3, SW1, SW2, U2
